File: EDA/TrailCurrentSwitchback/TrailCurrentSwitchback.kicad_sch (KiCad schematic)
At the start: 0 parts

Commit message: EDA for CAN Hat for waveshare relay and cad for milling pcb edges and drilling holes on Genmitsu 3030
Parts:
- added IC1: SN65HVD230DR, TrailCurrentFootprints:SN65HVD230DR, symbol TrailCurrentSymbolLibrary:SN65HVD230DR
- added J1, J2: Conn_01x20, Connector_PinSocket_2.54mm:PinSocket_1x20_P2.54mm_Vertical, symbol Connector_Generic:Conn_01x20
- added J3: S2B-XH-SM4-TB, TrailCurrentFootprints:JST_S2B-XH-SM4-TB, symbol TrailCurrentSymbolLibrary:S2B-XH-SM4-TB
- added R1: 10k, Resistor_SMD:R_1206_3216Metric_Pad1.30x1.75mm_HandSolder, symbol Device:R
Connections:
- new net: IC1.8 (RS), R1.2
- new net +3.3V: IC1.3 (VCC), J1.11 (Pin_11), J1.4 (Pin_4), J1.5 (Pin_5)
- new net CAN_H: IC1.7 (CANH), J3.2
- new net CAN_L: IC1.6 (CANL), J3.1
- new net CAN_RX: IC1.1 (D), J1.14 (Pin_14)
- new net CAN_TX: IC1.4 (R), J1.15 (Pin_15)
- new net GND: IC1.2 (GND), J1.13 (Pin_13), J1.18 (Pin_18), J1.3 (Pin_3), J1.8 (Pin_8), J2.13 (Pin_13), J2.18 (Pin_18), J2.3 (Pin_3), J2.8 (Pin_8), R1.1
- no-connect marks 0 -> 28
